Commit message: change urdf xacro to multiple xacro files with macros

File: m2wr_description/urdf/m2wr.xacro (robot description, xacro)
@@ -1,51 +1,8 @@
+<?xml version="1.0"?>
 <robot name="m2wr" xmlns:xacro="https://www.ros.org/wiki/xacro" >
-  <material name="black">
-    <color rgba="0.0 0.0 0.0 1.0"/>
-  </material>
-  <material name="blue">
-    <color rgba="0.203125 0.23828125 0.28515625 1.0"/>
-  </material>
-  <material name="green">
-    <color rgba="0.0 0.8 0.0 1.0"/>
-  </material>
-  <material name="grey">
-    <color rgba="0.2 0.2 0.2 1.0"/>
-  </material>
-  <material name="orange">
-    <color rgba="1.0 0.423529411765 0.0392156862745 1.0"/>
-  </material>
-  <material name="brown">
-    <color rgba="0.870588235294 0.811764705882 0.764705882353 1.0"/>
-  </material>
-  <material name="red">
-    <color rgba="0.80078125 0.12890625 0.1328125 1.0"/>
-  </material>
-  <material name="white">
-    <color rgba="1.0 1.0 1.0 1.0"/>
-  </material>
-  <gazebo reference="link_chassis">
-    <material>Gazebo/Orange</material>
-  </gazebo>
-  <gazebo reference="link_left_wheel">
-    <material>Gazebo/Blue</material>
-  </gazebo>
-  <gazebo reference="link_right_wheel">
-    <material>Gazebo/Blue</material>
-  </gazebo>
-  <gazebo>
-    <plugin filename="libgazebo_ros_diff_drive.so" name="differential_drive_controller">
-      <alwaysOn>true</alwaysOn>
-      <updateRate>20</updateRate>
-      <leftJoint>joint_left_wheel</leftJoint>
-      <rightJoint>joint_right_wheel</rightJoint>
-      <wheelSeparation>0.4</wheelSeparation>
-      <wheelDiameter>0.2</wheelDiameter>
-      <torque>0.1</torque>
-      <commandTopic>cmd_vel</commandTopic>
-      <odometryTopic>odom</odometryTopic>
-      <odometryFrame>odom</odometryFrame>
-      <robotBaseFrame>link_chassis</robotBaseFrame>
-    </plugin>
-  </gazebo>
+  <!--include the xacro files-->
+  <xacro:include filename="$(find m2wr_description)/urdf/materials.xacro" />
+  <xacro:include filename="$(find m2wr_description)/urdf/gazebo.xacro" />
+  <xacro:include filename="$(find m2wr_description)/urdf/macro.xacro" />
   <link name="link_chassis">
     <!-- pose and inertial -->
@@ -92,61 +49,37 @@
     </visual>
     </link>
-  <!-- Create wheel right -->
-  <link name="link_right_wheel">
+  <!-- Create wheel right link -->
+  <xacro:link_wheel name="link_right_wheel" />
+  <!--   Joint for right wheel  -->
+  <xacro:joint_wheel name="joint_right_wheel"  child="link_right_wheel"  origin_xyz="-0.05 0.15 0"  />
+  <!-- create Left Wheel link -->
+  <xacro:link_wheel name="link_left_wheel" />
+  <!--   Joint for left wheel  -->
+  <xacro:joint_wheel name="joint_left_wheel"   child="link_left_wheel"   origin_xyz="-0.05 -0.15 0" />
+  <link name="sensor_laser">
     <inertial>
-      <mass value="0.2"/>
-      <origin rpy="0 1.5707 1.5707" xyz="0 0 0"/>
-      <inertia ixx="0.00052666666" ixy="0" ixz="0" iyy="0.00052666666" iyz="0" izz="0.001"/>
+      <origin xyz="0 0 0" rpy="0 0 0" />
+      <mass value="1" />
+      <!-- RANDOM INERTIA BELOW -->
+      <inertia ixx="0.02" ixy="0" ixz="0" iyy="0.02" iyz="0" izz="0.02"/>
     </inertial>
-    <collision name="link_right_wheel_collision">
-      <origin rpy="0 1.5707 1.5707" xyz="0 0 0" />
+    <visual>
+      <origin xyz="0 0 0" rpy="0 0 0" />
       <geometry>
-        <cylinder length="0.04" radius="0.1"/>
+        <cylinder radius="0.05" length="0.1"/>
+      </geometry>
+      <material name="white" />
+    </visual>
+    <collision>
+      <origin xyz="0 0 0" rpy="0 0 0"/>
+      <geometry>
+        <cylinder radius="0.05" length="0.1"/>
       </geometry>
     </collision>
-    <visual name="link_right_wheel_visual">
-      <origin rpy="0 1.5707 1.5707" xyz="0 0 0"/>
-      <geometry>
-        <cylinder length="0.04" radius="0.1"/>
-      </geometry>
-    </visual>
   </link>
-  <!--   Joint for right wheel  -->
-  <joint name="joint_right_wheel" type="continuous">
-    <origin rpy="0 0 0" xyz="-0.05 0.15 0"/>
-    <child link="link_right_wheel" />
+  <joint name="joint_sensor_laser" type="fixed">
+    <origin xyz="0.15 0 0.05" rpy="0 0 0"/>
     <parent link="link_chassis"/>
-    <axis rpy="0 0 0" xyz="0 1 0"/>
-    <limit effort="10000" velocity="1000"/>
-    <joint_properties damping="1.0" friction="1.0" />
-  </joint>
-  <!-- Left Wheel link -->
-  <link name="link_left_wheel">
-    <inertial>
-      <mass value="0.2"/>
-      <origin rpy="0 1.5707 1.5707" xyz="0 0 0"/>
-      <inertia ixx="0.00052666666" ixy="0" ixz="0" iyy="0.00052666666" iyz="0" izz="0.001"/>
-    </inertial>
-    <collision name="link_left_wheel_collision">
-      <origin rpy="0 1.5707 1.5707" xyz="0 0 0" />
-      <geometry>
-        <cylinder length="0.04" radius="0.1"/>
-      </geometry>
-    </collision>
-    <visual name="link_left_wheel_visual">
-      <origin rpy="0 1.5707 1.5707" xyz="0 0 0"/>
-      <geometry>
-        <cylinder length="0.04" radius="0.1"/>
-      </geometry>
-    </visual>
-  </link>
-  <!--   Joint for right wheel  -->
-  <joint name="joint_left_wheel" type="continuous">
-    <origin rpy="0 0 0" xyz="-0.05 -0.15 0"/>
-    <child link="link_left_wheel" />
-    <parent link="link_chassis"/>
-    <axis rpy="0 0 0" xyz="0 1 0"/>
-    <limit effort="10000" velocity="1000"/>
-    <joint_properties damping="1.0" friction="1.0" />
+    <child link="sensor_laser"/>
   </joint>
 </robot>

Commit message: stack ur to the top surface of the robot, but the computer is too slow to simulate

File: m2wr_description/urdf/m2wr.xacro (robot description, xacro)
@@ -5,4 +5,12 @@
   <xacro:include filename="$(find m2wr_description)/urdf/gazebo.xacro" />
   <xacro:include filename="$(find m2wr_description)/urdf/macro.xacro" />
+  <!-- include the ur10e -->
+  <!--xacro:include filename="$(find ur_e_description)/urdf/ur10e.urdf.xacro"/>
+  <xacro:ur10e_robot prefix="" joint_limited="false"/>
+  <joint name="joint_ur" type="fixed">
+    <parent link="link_chassis" />
+    <child link = "base_link" />
+    <origin xyz="0.0 0.0 0.0" rpy="0.0 0.0 0.0" />
+  </joint-->
   <link name="link_chassis">
     <!-- pose and inertial -->
@@ -21,5 +29,5 @@
       <origin rpy="0 0 0" xyz="0 0 0"/>
       <geometry>
-        <box size="0.5 0.3 0.07"/>
+        <box size="1 0.6 0.15"/>
       </geometry>
       <material name="blue"/>
@@ -27,7 +35,7 @@
     <!-- caster front -->
     <collision name="caster_front_collision">
-      <origin rpy=" 0 0 0" xyz="0.35 0 -0.05"/>
+      <origin rpy=" 0 0 0" xyz="0.5 0 -0.08"/>
       <geometry>
-        <sphere radius="0.05"/>
+        <sphere radius="0.08"/>
       </geometry>
       <surface>
@@ -43,7 +51,7 @@
     </collision>
     <visual name="caster_front_visual">
-      <origin rpy=" 0 0 0" xyz="0.2 0 -0.05"/>
+      <origin rpy=" 0 0 0" xyz="0.4 0 -0.08"/>
       <geometry>
-        <sphere radius="0.05"/>
+        <sphere radius="0.08"/>
       </geometry>
     </visual>
@@ -52,9 +60,9 @@
   <xacro:link_wheel name="link_right_wheel" />
   <!--   Joint for right wheel  -->
-  <xacro:joint_wheel name="joint_right_wheel"  child="link_right_wheel"  origin_xyz="-0.05 0.15 0"  />
+  <xacro:joint_wheel name="joint_right_wheel"  child="link_right_wheel"  origin_xyz="-0.05 0.3 0"  />
   <!-- create Left Wheel link -->
   <xacro:link_wheel name="link_left_wheel" />
   <!--   Joint for left wheel  -->
-  <xacro:joint_wheel name="joint_left_wheel"   child="link_left_wheel"   origin_xyz="-0.05 -0.15 0" />
+  <xacro:joint_wheel name="joint_left_wheel"   child="link_left_wheel"   origin_xyz="-0.05 -0.3 0" />
   <link name="sensor_laser">
     <inertial>
@@ -79,5 +87,5 @@
   </link>
   <joint name="joint_sensor_laser" type="fixed">
-    <origin xyz="0.15 0 0.05" rpy="0 0 0"/>
+    <origin xyz="0.3 0 0.05" rpy="0 0 0"/>
     <parent link="link_chassis"/>
     <child link="sensor_laser"/>

File: m2wr_description/urdf/macro.xacro (robot description, xacro)
@@ -11,5 +11,5 @@
               <origin rpy="0 1.5707 1.5707" xyz="0 0 0"/>
               <geometry>
-                <cylinder length="0.04" radius="0.1"/>
+                <cylinder length="0.04" radius="0.2"/>
               </geometry>
             </collision>
@@ -17,5 +17,5 @@
               <origin rpy="0 1.5707 1.5707" xyz="0 0 0"/>
               <geometry>
-                <cylinder length="0.04" radius="0.1"/>
+                <cylinder length="0.04" radius="0.2"/>
               </geometry>
             </visual>

Commit message: add ur arm into the gazebo

File: m2wr_description/urdf/m2wr.xacro (robot description, xacro)
@@ -2,9 +2,10 @@
 <robot name="m2wr" xmlns:xacro="https://www.ros.org/wiki/xacro" >
   <!--include the xacro files-->
+  <xacro:include filename="$(find ur_e_description)/urdf/common.gazebo.xacro" />
   <xacro:include filename="$(find m2wr_description)/urdf/materials.xacro" />
   <xacro:include filename="$(find m2wr_description)/urdf/gazebo.xacro" />
   <xacro:include filename="$(find m2wr_description)/urdf/macro.xacro" />
   <!-- include the ur10e -->
-  <!--xacro:include filename="$(find ur_e_description)/urdf/ur10e.urdf.xacro"/>
+  <xacro:include filename="$(find ur_e_description)/urdf/ur10e.urdf.xacro"/>
   <xacro:ur10e_robot prefix="" joint_limited="false"/>
   <joint name="joint_ur" type="fixed">
@@ -12,5 +13,5 @@
     <child link = "base_link" />
     <origin xyz="0.0 0.0 0.0" rpy="0.0 0.0 0.0" />
-  </joint-->
+  </joint>
   <link name="link_chassis">
     <!-- pose and inertial -->
