Commit message: added sensor plugin and tested in rviz and gazebo

File: m2wr_description/urdf/gazebo.xacro (robot description, xacro)
@@ -10,4 +10,5 @@
     <material>Gazebo/Blue</material>
   </gazebo>
+  <!--differential drive controller plugin-->
   <gazebo>
     <plugin filename="libgazebo_ros_diff_drive.so" name="differential_drive_controller">
@@ -25,3 +26,35 @@
     </plugin>
   </gazebo>
+  <!-- sensor plugin -->
+  <gazebo reference="sensor_laser">
+    <sensor type="ray" name="head_hokuyo_sensor">
+      <pose>0 0 0 0 0 0</pose>
+      <visualize>false</visualize>
+      <update_rate>20</update_rate>
+      <ray>
+        <scan>
+          <horizontal>
+            <samples>720</samples>
+            <resolution>1</resolution>
+            <min_angle>-1.570796</min_angle>
+            <max_angle>1.570796</max_angle>
+          </horizontal>
+        </scan>
+        <range>
+          <min>0.10</min>
+          <max>10.0</max>
+          <resolution>0.01</resolution>
+        </range>
+        <noise>
+          <type>gaussian</type>
+          <mean>0.0</mean>
+          <stddev>0.01</stddev>
+        </noise>
+      </ray>
+      <plugin name="gazebo_ros_head_hokuyo_controller" filename="libgazebo_ros_laser.so">
+        <topicName>/m2wr/laser/scan</topicName>
+        <frameName>sensor_laser</frameName>
+      </plugin>
+    </sensor>
+  </gazebo>
 </robot>

File: m2wr_description/urdf/m2wr.xacro (robot description, xacro)
@@ -61,6 +61,6 @@
       <origin xyz="0 0 0" rpy="0 0 0" />
       <mass value="1" />
-      <!-- RANDOM INERTIA BELOW -->
-      <inertia ixx="0.02" ixy="0" ixz="0" iyy="0.02" iyz="0" izz="0.02"/>
+      <!-- calculate inertia from the macros -->
+      <xacro:cylinder_inertia mass="1" r="0.05" l="0.1" />
     </inertial>
     <visual>

File: m2wr_description/urdf/macro.xacro (robot description, xacro)
@@ -32,3 +32,7 @@
       </joint>
     </xacro:macro>
+    <xacro:macro name="cylinder_inertia" params="mass r l">
+        <inertia ixx="${mass*(3*r*r+l*l)/12}" ixy = "0" ixz = "0"
+	        iyy="${mass*(3*r*r+l*l)/12}" iyz = "0" izz="${mass*(r*r)/2}" />
+    </xacro:macro>
 </robot>

Commit message: change to 4 wheel base

File: m2wr_description/urdf/gazebo.xacro (robot description, xacro)
@@ -15,6 +15,6 @@
       <alwaysOn>true</alwaysOn>
       <updateRate>20</updateRate>
-      <leftJoint>joint_left_wheel</leftJoint>
-      <rightJoint>joint_right_wheel</rightJoint>
+      <leftJoint>joint_left_rear_wheel</leftJoint>
+      <rightJoint>joint_right_rear_wheel</rightJoint>
       <wheelSeparation>0.4</wheelSeparation>
       <wheelDiameter>0.2</wheelDiameter>

File: m2wr_description/urdf/m2wr.xacro (robot description, xacro)
@@ -24,5 +24,5 @@
     <collision name="collision_chassis">
       <geometry>
-        <box size="0.5 0.3 0.07"/>
+        <box size="1.0 0.3 0.07"/>
       </geometry>
     </collision>
@@ -59,11 +59,15 @@
     </link>
   <!-- Create wheel right link -->
-  <xacro:link_wheel name="link_right_wheel" />
+  <xacro:link_wheel name="link_right_front_wheel" />
+  <xacro:link_wheel name="link_right_rear_wheel" />
   <!--   Joint for right wheel  -->
-  <xacro:joint_wheel name="joint_right_wheel"  child="link_right_wheel"  origin_xyz="-0.05 0.3 0"  />
+  <xacro:joint_wheel name="joint_right_front_wheel"  child="link_right_front_wheel"  origin_xyz="0.5 0.3 0"  />
+  <xacro:joint_wheel name="joint_right_rear_wheel"  child="link_right_rear_wheel"  origin_xyz="-0.5 0.3 0"  />
   <!-- create Left Wheel link -->
-  <xacro:link_wheel name="link_left_wheel" />
+  <xacro:link_wheel name="link_left_front_wheel" />
+  <xacro:link_wheel name="link_left_rear_wheel" />
   <!--   Joint for left wheel  -->
-  <xacro:joint_wheel name="joint_left_wheel"   child="link_left_wheel"   origin_xyz="-0.05 -0.3 0" />
+  <xacro:joint_wheel name="joint_left_front_wheel"   child="link_left_front_wheel"   origin_xyz="0.5 -0.3 0" />
+  <xacro:joint_wheel name="joint_left_rear_wheel"  child="link_left_rear_wheel"   origin_xyz="-0.5 -0.3 0" />
   <link name="sensor_laser">
     <inertial>
